Commit message: visuals of cartpole

File: install/cartpole_sim/share/cartpole_sim/urdf/cartpole.urdf (robot description, URDF)
Before this commit: robot cartpole, 3 links, 2 joints
Links:
- link cart: geometry collision box size=0.4 0.2 0.1; visual box size=0.4 0.2 0.1
- link pole: geometry collision cylinder length=1.0 radius=0.03; visual cylinder length=1.0 radius=0.03
Joints:
- joint pole_joint: axis 0 0 1 -> 0 1 0
