Commit message: enabling wrench (to apply commands to robot from ros) via world enabling that (can't be done by urdf)

File: src/cartpole_sim/urdf/cartpole.urdf (robot description, URDF)
Before this commit: robot cartpole, 3 links, 2 joints
Links:
- removed link world
- added link base_link, mass 0.001; collision box size=0.01 0.01 0.01; visual box size=0.01 0.01 0.01
Joints:
- joint cart_joint: limit lower=-2 upper=2 effort=50 velocity=5 -> lower=-2 upper=2 effort=100 velocity=5; origin (none) -> xyz=0 0 0; parent world -> base_link
- joint pole_joint: origin (none) -> xyz=0 0 0.1
